File: hardware/kicad/c64_usb_keyboard.kicad_sch (KiCad schematic)
At the start: 0 parts

Commit message: Migrate to Raspberry Pi Pico 2 (RP2350): 5V-tolerant native open-drain matrix, KiCad 8 project fix, and ultra-simplified BOM
Other:
- title: C64 USB Keyboard & Wireless Host Adapter (DIP/THT) -> C64 USB Keyboard & Wireless Host Adapter (Pico 2 / RP2350)
Changed lines of the file:
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@@
 (kicad_sch
-  (version 20230121)
-  (generator "eeschema")
-  (generator_version "7.0")
-  (paper "A4")
-  (title_block
-    (title "C64 USB Keyboard & Wireless Host Adapter (DIP/THT)")
-    (date "2026-09-30")
-    (rev "v1.0")
-    (company "AGRAVITY Hardware / Software Project")
-    (comment 1 "Raspberry Pi Pico + 74HCT245 + BAT42 Schottky + Voltage Dividers")
-    (comment 2 "100% DIP and THT Construction - C64 CN8 Connector")
-  )
-  (sheet_instances
-    (path "/"
-      (page "1")
-    )
-  )
+	(version 20231120)
+	(generator "eeschema")
+	(generator_version "8.0")
+	(paper "A4")
+	(title_block
+		(title "C64 USB Keyboard & Wireless Host Adapter (Pico 2 / RP2350)")
+		(date "2026-10-01")
+		(rev "v2.0 - Pico 2 Ultra-Simplified")
+		(company "AGRAVITY Hardware / Software Project")
+		(comment 1 "RP2350 5V-Tolerant GPIOs + Native Open-Drain Matrix Emulation")
+		(comment 2 "Direct C64 Motherboard CN8 Interface - Zero Level Shifter ICs")
+	)
+	(sheet_instances
+		(path "/"
+			(page "1")
+		)
+	)
 )
